File: Adaptadores/Microchip/ARE_adaptadora_dsPIC-PIC32_64pin.sch (EAGLE design)
At the start: 89 parts, among them IC1 PIC32MX, IC2 12F, IC3 PIC24FJ32GA004, IC4 PIC16F1517/19PT, IC5 16F, IC6 10F, U2 STM32-M-64-LQFP

Commit message: New version and a massive re-arrengement
New version of base trainer. Now it is called Ardu-Trainer MultiMicro,
as it has an ATMEGA32U4 with all its pins available. It can be
programmed with Arduino bootloader or directly with your own firmware.
All of MultiMicro adapters have been revised, cleaned and sorted.
Parts:
- removed C10, C11, C12, C15, C16, C17, C18, C19, C22, C24, C27, C28, C32, C35, C36: 100n, rcl:C-EUC0805
- removed C13, C14, C20, C21, C29, C30, C33, C34: 18p, rcl:C-EUC0805
- removed C23: 1u, rcl:C-EUC0805
- removed C25, C9: 10uF, rcl:CPOL-EUSMCC
- removed IC2: 12F, ic-package:DIL8S
- removed IC3: PIC24FJ32GA004, microchip:PIC24FJ32GA004
- removed IC4: PIC16F1517/19PT, microchip:PIC16F1517/19PT
- removed IC5: 16F, ic-package:DIL14S
- removed IC6: 10F, ic-package:DIL8S
- removed JP1, JP2, JP3: (no value), SparkFun:M05PTH
- removed LED2, LED3, LED4, LED5: (no value), led:LEDCHIPLED_0805
- removed Q2, Q3, Q4, Q6: (no value), crystal:CRYSTALHC18U-V
- removed R3, R6, R8: 4K7, rcl:R-EU_R0805
- removed R4, R5, R7, R9: 1K, rcl:R-EU_R0805
- removed S2, S3, S4, S5: (no value), switch-omron:10-XX
- removed SJ1, SJ2: (no value), jumper:SJ2W
- removed SJ3: (no value), jumper:SJ
- removed SV10, SV11, SV12, SV4, SV5, SV6, SV7, SV8, SV9: (no value), con-lsta:FE10-2W
- removed U$3: FE02-2W, con-lsta:FE02-2W
- removed U2: STM32-M-64-LQFP, pel_stm32:STM32-M-64-LQFP
- added JMP2: 0R-JUMPA, jump-0r-smd:0R-JUMPA
Connections:
- removed net N$14: IC6.6
- removed net N$2: LED2.A, R4.1
- removed net N$3: LED3.A, R5.1
- removed net N$4: LED4.A, R7.1
- removed net N$6: SV7.11
- removed net N$7: SV7.9
- removed net N$8: LED5.A, R9.1
- removed net N$9: IC6.1
- removed net P201: IC3.RA4, SV4.1
- removed net P203: IC3.RC3, SV4.3
- removed net P204: IC3.TDI, SV4.4
- removed net P205: IC3.RC5, SV4.5
- removed net P206: IC3.RC4, SV4.6
- removed net P207: IC3.RB6, SV4.7
- removed net P208: IC3.RB5, SV4.8
- removed net P209: IC3.RB8, SJ1.1, SV4.9
- removed net P210: IC3.RB7, SV4.10
- removed net P211: IC3.RC6, SV4.11
- removed net P212: IC3.RB9, SJ2.3, SV4.12
- removed net P213: IC3.RC8, SV4.13
- removed net P214: IC3.RC7, SV4.14
- removed net P215: IC3.RB10, SV4.15
- removed net P216: IC3.RC9, SV4.16
- removed net P217: IC3.RB12, SV4.17
- removed net P218: IC3.RB11, SV4.18
- removed net P219: IC3.TMS, SV4.19
- removed net P220: IC3.RB13, SV4.20
- removed net P221: IC3.RB14, SV5.1
- removed net P222: IC3.TCK, SV5.2
- removed net P223: IC3.RA0, SV5.3
- removed net P224: IC3.RB15, SV5.4
- removed net P225: IC3.RB0, SJ1.3, SV5.5
- removed net P226: IC3.RA1, SV5.6
- removed net P227: IC3.RB2, SV5.7
- removed net P228: IC3.RB1, SJ2.1, SV5.8
- removed net P229: IC3.RC0, SV5.9
- removed net P230: IC3.RB3, SV5.10
- removed net P231: IC3.RC2, SV5.11
- removed net P232: IC3.RC1, SV5.12
- removed net P235: IC3.RB4, SV5.15
- removed net P236: IC3.TDO, SV5.16
- removed net P2GC: JP1.5, SJ2.2
- removed net P2GD: JP1.4, SJ1.2
- removed net P2MCLR: IC3.!MCLR, JP1.1, R3.1, S2.S, SV4.2
- removed net P2OSC1: C13.1, IC3.RA2, Q2.2, SV5.14
- removed net P2OSC2: C14.1, IC3.RA3, Q2.1, SV5.13
- removed net P302: SV6.19, U2.PB9-TIM4CH4-I2C1SDA/CANTX
- removed net P303: SV6.20, U2.PB8-TIM4CH3-I2C1SCL/CANRX
- removed net P305: SV6.17, U2.BOOT0
- removed net P306: SV6.18, U2.PB7-I2C1SDA/TIM4CH2-USART1RX
- removed net P308: SV6.15, U2.PB6-I2C1SCL/TIM4CH1-USART1TX
- removed net P309: SV6.16, U2.PB5-I2C1SMBAI-TIM3CH2/SPI1MOSI
- removed net P311: SV6.13, U2.PB4/JNTRST--TIM3CH1/SPI1MISO
- removed net P312: SV6.14, U2.PB3/JTDO--TIM2CH2/TRACESWO/SPI1SCK
- removed net P314: SV6.11, U2.PD2-TIM3ETR
- removed net P315: SV6.12, U2.PC12--USART3CK
- removed net P317: SV6.9, U2.PC11--USART3RX
- removed net P318: SV6.10, U2.PC10--USART3TX
- removed net P320: SV6.7, U2.PA15/JTDI-TIM2CH1ETR/SPI1NSS
- removed net P321: SV6.8, U2.PA14/JTCK/SWCLK
- removed net P323: SV6.5, U2.PA13/JTMS/SWDIO
- removed net P324: SV6.6, U2.PA12-USART1RTS/CANTX/USBDP/TIM1ETR
- removed net P326: SV6.3, U2.PA11-USART1CTS/CANRX/USBDM/TIM1CH4
- removed net P327: SV6.4, U2.PA10-USART1RX/TIM1CH3
- removed net P329: SV6.1, U2.PA9-USART1TX/TIM1CH2
- removed net P330: SV6.2, U2.PA8-USART1CK/MCO/TIM1CH1
- removed net P332: SV7.19, U2.PC9-TIM3CH4
- removed net P333: SV7.20, U2.PC8-TIM3CH3
- removed net P335: SV7.17, U2.PC7-TIM3CH2
- removed net P336: SV7.18, U2.PC6-TIM3CH1
- removed net P338: SV7.15, U2.PB15-SPI2MOSI/TIM1CH3N
- removed net P339: SV7.16, U2.PB14-SPI2MISO/USART3RTS/TIM1CH2N
- removed net P341: SV7.13, U2.PB13-SPI2SCK/USART3CTS/TIM1CH1N
- removed net P342: SV7.14, U2.PB12-SPI2NSS/I2C2SMBAI/USART3CK/TIM1BKIN
- removed net P350: SV7.3, SV7.7, U2.PB10-I2C2SCL/USART3TX-TIM2CH3
- removed net P351: SV7.8, U2.PB11-I2C2SDA/USART3RX-TIM2CH4
- removed net P353: SV7.1, U2.PB1-ADC9/TIM3CH4-TIM1CH3N
- removed net P354: SV7.6, U2.PB2/BOOT1
- removed net P356: SV8.19, U2.PC5-ADC15
- removed net P357: SV7.4, U2.PB0-ADC8/TIM3CH3-TIM1CH2N
- removed net P359: SV8.17, U2.PA7-SPI1MOSI/ADC7/TIM3CH2-TIM1CH1N
- removed net P360: SV7.2, U2.PC4-ADC14
- removed net P362: SV8.15, U2.PA5-SPI1SCK/ADC5
- removed net P363: SV8.20, U2.PA6-SPI1MISO/ADC6/TIM3CH1-TIM1BKIN
- removed net P365: SV8.13, U2.PA3-USART2RX/ADC3/TIM2CH4
- removed net P366: SV8.18, U2.PA4-SPI1NSS/ADC4/USART2CK
- removed net P368: SV8.11, U2.PA1-USART2RTS/ADC1/TIM2CH2
- removed net P369: SV8.16, U2.PA2-USART2TX/ADC2/TIM2CH3
- removed net P371: SV8.9, U2.PC3-ADC13
- removed net P372: SV8.14, U2.PA0-WKUP/USART2CTS/ADC0/TIM2CH1ETR
- removed net P374: SV8.7, U2.PC1-ADC11
- removed net P375: SV8.12, U2.PC2-ADC12
- removed net P378: SV8.10, U2.PC0-ADC10
- removed net P380: SV8.3, U2.PC15-OSC32_OUT
- removed net P383: SV8.1, U2.PC13-TAMPER-RTC
- removed net P384: SV8.6, U2.PC14-OSC32_IN
- removed net P387: SV8.4
- removed net P3MCLR: C19.1, S3.S, SV8.2, U2.NRST
- removed net P3OSC1: C20.1, Q3.2, SV8.8, U2.PD0-OSC_IN-CANRX
- removed net P3OSC2: C21.1, Q3.1, SV8.5, U2.PD1-OSC_OUT-CANTX
- removed net P401: IC4.RC1/SOSCI/CCP2, SV9.1
- removed net P403: IC4.RC3/AN15/SCK/SCL, SV9.3
- removed net P404: IC4.RC2/AN14/CCP1, SV9.4
- removed net P405: IC4.RD1/AN21, SV9.5
- removed net P406: IC4.RD0/AN20, SV9.6
- removed net P407: IC4.RD3/AN23, SV9.7
- removed net P408: IC4.RD2/AN22, SV9.8
- removed net P409: IC4.RC5/AN17/SDO, SV9.9
- removed net P410: IC4.RC4/AN16/SDI/SDA, SV9.10
- removed net P411: IC4.DT/RX/AN19/RC7, SV9.11
- removed net P412: IC4.RC6/AN18/TX/CK, SV9.12
- removed net P413: IC4.AN25/RD5, SV9.13
- removed net P414: IC4.AN24/RD4, SV9.14
- removed net P415: IC4.AN27/RD7, SV9.15
- removed net P416: IC4.AN26/RD6, SV9.16
- removed net P417: IC4.AN10/RB1, SV9.17
- removed net P418: IC4.INT/AN12/RB0, SV9.18
- removed net P419: IC4.CCP2/AN9/RB3, SV9.19
- removed net P420: IC4.AN8/RB2, SV9.20
- removed net P421: IC4.AN11/RB4, SV10.1
- removed net P422: IC4.T1G/AN13/RB5, SV10.2
- removed net P425: IC4.!SS!/AN0/RA0, SV10.5
- removed net P426: IC4.AN1/RA1, SV10.6
- removed net P427: IC4.AN2/RA2, SV10.7
- removed net P428: IC4.VREF+/AN3/RA3, SV10.8
- removed net P429: IC4.RA4/TOCKI, SJ3.2, SV10.9
- removed net P430: IC4.RA5/AN4/!SS!/VCAP, SV10.10
- removed net P431: IC4.RE0/AN5, SV10.11
- removed net P432: IC4.RE1/AN6, SV10.12
- removed net P433: IC4.RE2/AN7, SV10.13
- removed net P436: IC4.RC0/SOSCO/T1CKI, SV10.16
- removed net P4GC: IC4.ICDCLK/ICSPCLK/RB6, JP2.5, SV10.3
- removed net P4GD: IC4.ICDDAT/ICSPDAT/RB7, JP2.4, SV10.4
- removed net P4MCLR: IC4.VPP/!MCLR!/RE3, JP2.1, R6.1, S4.S, SV9.2
- removed net P4OSC1: C29.1, IC4.RA7/OSC1/CLKIN, Q4.2, SV10.14
- removed net P4OSC2: C30.1, IC4.RA6/OSC2/CLKOUT, Q4.1, SV10.15
- removed net P502: SV11.2
- removed net P504: SV11.4
- removed net P506: SV11.6
- removed net P507: IC6.3, SV11.7
- removed net P508: SV11.8
- removed net P513: IC2.5, SV11.13
- removed net P514: SV11.14
- removed net P516: SV11.16
- removed net P517: IC2.3, SV11.17
- removed net P518: IC2.2, SV11.18
- removed net P521: IC5.8, SV12.1
- removed net P522: IC5.7, SV12.2
- removed net P523: IC5.9, SV12.3
- removed net P524: IC5.6, SV12.4
- removed net P525: IC5.10, SV12.5
- removed net P526: IC5.5, SV12.6
- removed net P527: IC5.11, SV12.7
- removed net P533: SV12.13
- removed net P534: SV12.14
- removed net P535: SV12.15
- removed net P536: SV12.16
- removed net P5GC: IC2.6, IC5.12, IC6.4, JP3.5, SV11.11, SV11.5, SV12.9
- removed net P5GD: IC2.7, IC5.13, IC6.5, JP3.4, SV11.12, SV11.3, SV12.11
- removed net P5MCLR: IC2.4, IC5.4, IC6.8, JP3.1, R8.1, S5.S, SV11.1, SV11.15, SV12.8
- removed net P5OSC1: C33.1, IC5.2, Q6.2, SV12.12
- removed net P5OSC2: C34.1, IC5.3, Q6.1, SV12.10
- new net VREG: IC1.VREG, JMP2-0R.2
- net VCC: now also JMP2-0R.1; no longer C10.1, C11.1, C12.1, C15.1, C16.1, C17.1, C18.1, C22.1, C23.1, C24.1, C25.+, C27.1, C28.1, C32.1, C35.1, C36.1, C9.+, IC1.VREG, IC2.1, IC3.AVDD, IC3.VDD@1, IC3.VDD@2, IC3.VDDCORE, IC4.VDD, IC4.VDD@1, IC5.1, IC6.2, JP1.2, JP2.2, JP3.2, R3.2, R4.2, R5.2, R6.2, R7.2, R8.2, R9.2, SJ3.1, SV10.17, SV10.18, SV11.10, SV11.19, SV11.20, SV11.9, SV12.17, SV12.18, SV5.17, SV5.18, SV7.10, SV7.12, SV7.5, U$3.P$1, U$3.P$2, U2.VBAT, U2.VDD1, U2.VDD2, U2.VDD3, U2.VDD4, U2.VDDA
- net VSS: now also JMP2-0R.3; no longer C10.2, C11.2, C12.2, C13.2, C14.2, C15.2, C16.2, C17.2, C18.2, C19.2, C20.2, C21.2, C22.2, C23.2, C24.2, C25.-, C27.2, C28.2, C29.2, C30.2, C32.2, C33.2, C34.2, C35.2, C36.2, C9.-, IC2.8, IC3.AVSS, IC3.DISVREG, IC3.VSS@1, IC3.VSS@2, IC4.VSS, IC4.VSS@1, IC5.14, IC6.7, JP1.3, JP2.3, JP3.3, LED2.C, LED3.C, LED4.C, LED5.C, S2.P, S3.P, S4.P, S5.P, SV10.19, SV10.20, SV12.19, SV12.20, SV5.19, SV5.20, U$3.P$3, U$3.P$4, U2.VSS1, U2.VSS2, U2.VSS3, U2.VSS4, U2.VSSA
